File: PCB/keyboard.kicad_pcb (KiCad board)
At the start: 2 copper layers, 290.9 x 123.4 mm, 155 parts, among them SW1 SW_Push, SW10 SW_Push, SW11 SW_Push, SW12 SW_Push, SW13 SW_Push, SW14 SW_Push, SW15 SW_Push, SW16 SW_Push, SW17 SW_Push, SW18 SW_Push, SW19 SW_Push, SW2 SW_Push, SW20 SW_Push, SW21 SW_Push, SW22 SW_Push, SW23 SW_Push, SW24 SW_Push, SW25 SW_Push, SW26 SW_Push, SW27 SW_Push, SW28 SW_Push, SW29 SW_Push, SW3 SW_Push, SW30 SW_Push, SW31 SW_Push, SW32 SW_Push, SW33 SW_Push, SW34 SW_Push, SW35 SW_Push, SW36 SW_Push, SW37 SW_Push, SW38 SW_Push, SW39 SW_Push, SW4 SW_Push, SW40 SW_Push, SW41 SW_Push, SW42 SW_Push, SW43 SW_Push, SW44 SW_Push, SW45 SW_Push, SW46 SW_Push, SW47 SW_Push, SW48 SW_Push, SW49 SW_Push, SW5 SW_Push, SW50 SW_Push, SW51 SW_Push, SW52 SW_Push, SW53 SW_Push, SW54 SW_Push, SW55 SW_Push, SW56 SW_Push, SW57 SW_Push, SW58 SW_Push, SW59 SW_Push, SW6 SW_Push, SW60 SW_Push, SW61 SW_Push, SW62 RotaryEncoder_Switch, SW63 RotaryEncoder_Switch, SW7 SW_Push, SW8 SW_Push, SW9 SW_Push, U1 Pico

Commit message: updated PCB
Parts:
- removed D65, D66: LED_Small, LED_THT:LED_D5.0mm
- removed the G*** at (306.0, 106.2)
- removed the G*** at (226.8, 206.5)
- removed the G*** at (167.0, 206.2)
- removed the G*** at (311.8, 146.6)
- removed the G*** at (134.6, 105.4)
- removed the G*** at (271.7, 180.2)
- removed the G*** at (300.6, 184.2)
- removed the G*** at (146.4, 150.1)
- removed the G*** at (101.3, 144.8)
- removed the G*** at (192.4, 164.1)
- removed the G*** at (333.5, 106.2)
- removed the G*** at (266.6, 104.9)
- removed the G*** at (79.3, 193.1)
- removed the G*** at (199.0, 102.8)
- removed the G*** at (239.2, 133.9)
- removed the G*** at (335.0, 191.9)
- removed R1, R2, R3: 330Ω, Resistor_THT:R_Axial_DIN0309_L9.0mm_D3.2mm_P20.32mm_Horizontal
- added D73: 1N4148, Diode_THT:D_DO-35_SOD27_P7.62mm_Horizontal, B.Cu at (185.7, 111.7)
- added D74: 1N4148, Diode_THT:D_DO-35_SOD27_P7.62mm_Horizontal, B.Cu at (204.9, 111.7)
- added D75: 1N4148, Diode_THT:D_DO-35_SOD27_P7.62mm_Horizontal, B.Cu at (223.8, 111.6)
- added D76: 1N4148, Diode_THT:D_DO-35_SOD27_P7.62mm_Horizontal, B.Cu at (242.9, 111.6)
- added D77: 1N4148, Diode_THT:D_DO-35_SOD27_P7.62mm_Horizontal, B.Cu at (273.8, 112.0)
- added D78: 1N4148, Diode_THT:D_DO-35_SOD27_P7.62mm_Horizontal, B.Cu at (292.8, 112.0)
- added D79: 1N4148, Diode_THT:D_DO-35_SOD27_P7.62mm_Horizontal, B.Cu at (311.9, 112.0)
- added D80: 1N4148, Diode_THT:D_DO-35_SOD27_P7.62mm_Horizontal, B.Cu at (331.0, 111.8)
- added G***: LOGO, LOGO, F.Cu at (219.8, 154.2)
- added G***: LOGO, LOGO, B.Cu at (219.5, 154.2)
- added SW64: SW_Push, Button_Switch_Keyboard:SW_Cherry_MX_1.00u_PCB, F.Cu at (362.0, 199.3)
- added SW67: SW_Push, Button_Switch_Keyboard:SW_Cherry_MX_1.00u_PCB, F.Cu at (343.1, 180.2)
- added SW68: SW_Push, Button_Switch_Keyboard:SW_Cherry_MX_1.00u_PCB, F.Cu at (76.4, 102.1)
- added SW69: SW_Push, Button_Switch_Keyboard:SW_Cherry_MX_1.00u_PCB, F.Cu at (109.7, 102.1)
- added SW70: SW_Push, Button_Switch_Keyboard:SW_Cherry_MX_1.00u_PCB, F.Cu at (128.7, 102.1)
- added SW71: SW_Push, Button_Switch_Keyboard:SW_Cherry_MX_1.00u_PCB, F.Cu at (147.8, 102.1)
- added SW72: SW_Push, Button_Switch_Keyboard:SW_Cherry_MX_1.00u_PCB, F.Cu at (166.8, 102.1)
- added SW73: SW_Push, Button_Switch_Keyboard:SW_Cherry_MX_1.00u_PCB, F.Cu at (197.8, 102.1)
- added SW74: SW_Push, Button_Switch_Keyboard:SW_Cherry_MX_1.00u_PCB, F.Cu at (216.9, 102.1)
- added SW75: SW_Push, Button_Switch_Keyboard:SW_Cherry_MX_1.00u_PCB, F.Cu at (235.9, 102.1)
- added SW76: SW_Push, Button_Switch_Keyboard:SW_Cherry_MX_1.00u_PCB, F.Cu at (255.0, 102.1)
- added SW77: SW_Push, Button_Switch_Keyboard:SW_Cherry_MX_1.00u_PCB, F.Cu at (285.9, 102.1)
- added SW78: SW_Push, Button_Switch_Keyboard:SW_Cherry_MX_1.00u_PCB, F.Cu at (305.0, 102.1)
- added SW79: SW_Push, Button_Switch_Keyboard:SW_Cherry_MX_1.00u_PCB, F.Cu at (324.0, 102.1)
- added SW80: SW_Push, Button_Switch_Keyboard:SW_Cherry_MX_1.00u_PCB, F.Cu at (343.1, 102.1)
- D64, D67, D68, D69, D70, D71, D72: value LED_Small -> 1N4148; footprint LED_THT:LED_D5.0mm -> Diode_THT:D_DO-35_SOD27_P7.62mm_Horizontal; moved to B.Cu
- SW53: footprint Button_Switch_Keyboard:SW_Cherry_MX_2.75u_PCB -> Button_Switch_Keyboard:SW_Cherry_MX_1.75u_PCB
- SW60, SW61: footprint Button_Switch_Keyboard:SW_Cherry_MX_1.25u_PCB -> Button_Switch_Keyboard:SW_Cherry_MX_1.00u_PCB
- moved U1 276.3 mm to (362.8, 120.2), turned to 0 degrees
- moved D64 161.9 mm to (350.0, 208.3), turned to 90 degrees
- moved D68 135.3 mm to (64.3, 112.3), turned to 90 degrees
- moved D70 133.1 mm to (116.5, 112.0), turned to 90 degrees
- moved D67 126.0 mm to (331.0, 190.0), turned to 90 degrees
- moved SW62 104.1 mm to (359.4, 188.2), turned to 90 degrees
- moved D62 86.5 mm to (371.5, 177.3), turned to -90 degrees
- moved D71 76.5 mm to (135.7, 111.8), turned to 90 degrees
- moved SW63 71.3 mm to (359.4, 166.8), turned to 90 degrees
- moved D69 63.8 mm to (97.5, 112.1), turned to 90 degrees
- moved D63 53.5 mm to (371.5, 155.8), turned to -90 degrees
- moved D72 20.3 mm to (154.9, 111.6), turned to 90 degrees
- moved SW53 9.66 mm to (316.9, 180.2)
- moved D60 9.17 mm to (311.6, 209.2)
- moved SW60 6.96 mm to (323.9, 199.3)
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Connections:
- D64 pad 1: Net-(D64-K) -> row5
- D64 pad 2: red_anode -> Net-(D64-A)
- D67 pad 1: Net-(D67-K) -> row4
- D67 pad 2: blue_anode -> Net-(D67-A)
- D68 pad 1: Net-(D67-K) -> row6
- D68 pad 2: blue_anode -> Net-(D68-A)
- D69 pad 1: Net-(D67-K) -> row6
- D69 pad 2: blue_anode -> Net-(D69-A)
- D70 pad 1: Net-(D70-K) -> row6
- D70 pad 2: green_anode -> Net-(D70-A)
- D71 pad 1: Net-(D70-K) -> row6
- D71 pad 2: green_anode -> Net-(D71-A)
- D72 pad 1: Net-(D70-K) -> row6
- D72 pad 2: green_anode -> Net-(D72-A)
- U1 pad 25: re1 -> row6
- U1 pad 31: green_anode -> re1
- U1 pad 32: red_anode -> unconnected-(U1-GPIO27_ADC1-Pad32)
- U1 pad 34: blue_anode -> unconnected-(U1-GPIO28_ADC2-Pad34)
Routing:
- net row6: track 0.00 -> 320.2 mm
- net col1: track 106.6 -> 390.0 mm
- net GND: track 404.7 -> 165.2 mm, vias 6 -> 1
- net col2: track 140.1 -> 373.0 mm
- net col14: track 307.4 -> 87.6 mm
- net green_anode: track 197.7 -> 0.00 mm, vias 2 -> 0
- net col3: track 159.8 -> 356.9 mm
- net re3: track 236.5 -> 42.1 mm
- net re4: track 240.1 -> 50.9 mm, vias 0 -> 2
- net blue_anode: track 173.3 -> 0.00 mm, vias 2 -> 0
- net col4: track 195.7 -> 365.0 mm
- net red_anode: track 156.0 -> 0.00 mm, vias 4 -> 0
- net col5: track 265.7 -> 408.3 mm
- net col9: track 220.2 -> 349.6 mm
- net re2: track 205.6 -> 78.6 mm, vias 3 -> 0
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Other:
- board size 290.9 x 123.4 mm -> 314.9 x 121 mm
